Commit message: Update hokuyo.urdf.xacro
lower lidar position to costmap max height

File: src/turtlebot/turtlebot_description/urdf/sensors/hokuyo.urdf.xacro (robot description, xacro)
@@ -25,5 +25,5 @@
     <joint name="hokuyo_joint" type="fixed">
       <!--<axis xyz="0 0 1" />-->
-      <origin xyz="0.08 0 0.430" rpy="0 0 0"/>
+      <origin xyz="0.08 0 0.16" rpy="0 0 0"/>
       <parent link="${parent}"/>
       <child link="hokuyo_link"/>
